File: KiCAD/SNAC Sniffer/SNAC Sniffer Indent.sch (KiCad schematic (older format))
At the start: 11 parts, among them J1 PinHeader, J2 PinHeader, J3 PinHeader, J4 PinHeader, J5 PinHeader, J6 PinHeader, J7 PinHeader, J8 PinHeader, P1 HDMI_Female, P2 HDMI_Female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

Commit message: add ver.L
Parts:
- U1: footprint SNAC Sniffer:Arduino_Nano -> SNAC Sniffer:Arduino_Nano_Less_Pins
Changed lines of the file:
@@
 F 0 "U1" V 5304 5380 50  0000 L CNN
 F 1 "Arduino_Nano" V 5395 5380 50  0000 L CNN
-F 2 "SNAC Sniffer:Arduino_Nano" H 5350 4550 50  0001 L BNN
+F 2 "SNAC Sniffer:Arduino_Nano_Less_Pins" H 5350 4550 50  0001 L BNN
 F 3 "" H 5350 4550 50  0001 L BNN
 F 4 "Manufacturer Recommendations" H 5350 4550 50  0001 L BNN "STANDARD"
